File: pcb/transcoder.kicad_sch (KiCad schematic)
At the start: 35 parts, among them J1 MD-90SM, J2 Connector_RCA_2x3_REB, U1 BA7230LS, U2 LM1881, U3 THS7374

Commit message: Update
Connections:
- net B_IN: no longer C3.2, U1.15 (AB)
- net CVID_IN: no longer C4.2, U2.2 (C_IN)
- net G_IN: no longer C2.2, U1.14 (AG)
- net LAUD: now also J2.6 (Audio_Left); no longer J2.4 (L)
- net PB_OUT: now also J2.3 (Pb); no longer J2.2 (Pb)
- net PR_OUT: now also J2.1 (Pr); no longer J2.3 (Pr)
- net RAUD: now also J2.4 (Audio_Right); no longer J2.5 (R)
- net R_IN: no longer C1.2, U1.13 (AR)
- net Y_OUT: now also J2.5 (Y); no longer J2.1 (Y)
- new net B: C3.2, U1.15 (AB)
- new net CVID: C4.2, U2.2 (C_IN)
- new net G: C2.2, U1.14 (AG)
- new net R: C1.2, U1.13 (AR)
Changed lines of the file:
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@@
   (no_connect (at 123.19 102.87))
   (no_connect (at 198.12 121.92))
+  (no_connect (at 198.12 39.37))
   (no_connect (at 48.26 48.26))
   (no_connect (at 123.19 120.65))
@@
   (no_connect (at 93.98 123.19))
   (no_connect (at 123.19 107.95))
-  (no_connect (at 198.12 54.61))
   (no_connect (at 97.79 46.99))
   (no_connect (at 93.98 105.41))
@@
     (effects (font (size 1.27 1.27)) (justify right bottom))
   )
-  (label "PB_OUT" (at 198.12 39.37 180) (fields_autoplaced)
+  (label "PB_OUT" (at 198.12 43.18 180) (fields_autoplaced)
     (effects (font (size 1.27 1.27)) (justify right bottom))
   )
@@
     (effects (font (size 1.27 1.27)) (justify right bottom))
   )
-  (label "B_IN" (at 93.98 113.03 180) (fields_autoplaced)
+  (label "B" (at 93.98 113.03 180) (fields_autoplaced)
     (effects (font (size 1.27 1.27)) (justify right bottom))
   )
@@
     (effects (font (size 1.27 1.27)) (justify left bottom))
   )
-  (label "RAUD" (at 198.12 50.8 180) (fields_autoplaced)
+  (label "RAUD" (at 198.12 46.99 180) (fields_autoplaced)
     (effects (font (size 1.27 1.27)) (justify right bottom))
   )
@@
     (effects (font (size 1.27 1.27)) (justify left bottom))
   )
-  (label "PR_OUT" (at 198.12 43.18 180) (fields_autoplaced)
+  (label "PR_OUT" (at 198.12 35.56 180) (fields_autoplaced)
     (effects (font (size 1.27 1.27)) (justify right bottom))
   )
@@
     (effects (font (size 1.27 1.27)) (justify left bottom))
   )
-  (label "CVID_IN" (at 60.96 121.92 0) (fields_autoplaced)
+  (label "CVID" (at 60.96 121.92 0) (fields_autoplaced)
     (effects (font (size 1.27 1.27)) (justify left bottom))
   )
@@
     (effects (font (size 1.27 1.27)) (justify right bottom))
   )
-  (label "G_IN" (at 123.19 110.49 0) (fields_autoplaced)
-    (effects (font (size 1.27 1.27)) (justify left bottom))
-  )
-  (label "CVID_IN" (at 97.79 44.45 180) (fields_autoplaced)
-    (effects (font (size 1.27 1.27)) (justify right bottom))
-  )
-  (label "GND" (at 198.12 58.42 180) (fields_autoplaced)
-    (effects (font (size 1.27 1.27)) (justify right bottom))
-  )
-  (label "Y_OUT" (at 198.12 35.56 180) (fields_autoplaced)
-    (effects (font (size 1.27 1.27)) (justify right bottom))
-  )
-  (label "R_IN" (at 93.98 110.49 180) (fields_autoplaced)
+  (label "G" (at 123.19 110.49 0) (fields_autoplaced)
+    (effects (font (size 1.27 1.27)) (justify left bottom))
+  )
+  (label "CVID" (at 97.79 44.45 180) (fields_autoplaced)
+    (effects (font (size 1.27 1.27)) (justify right bottom))
+  )
+  (label "GND" (at 207.01 64.77 270) (fields_autoplaced)
+    (effects (font (size 1.27 1.27)) (justify right bottom))
+  )
+  (label "Y_OUT" (at 198.12 50.8 180) (fields_autoplaced)
+    (effects (font (size 1.27 1.27)) (justify right bottom))
+  )
+  (label "R" (at 93.98 110.49 180) (fields_autoplaced)
     (effects (font (size 1.27 1.27)) (justify right bottom))
   )
@@
     (effects (font (size 1.27 1.27)) (justify left bottom))
   )
-  (label "G_IN" (at 60.96 101.6 0) (fields_autoplaced)
+  (label "G" (at 60.96 101.6 0) (fields_autoplaced)
     (effects (font (size 1.27 1.27)) (justify left bottom))
   )
@@
     (effects (font (size 1.27 1.27)) (justify left bottom))
   )
-  (label "LAUD" (at 198.12 46.99 180) (fields_autoplaced)
+  (label "LAUD" (at 198.12 54.61 180) (fields_autoplaced)
     (effects (font (size 1.27 1.27)) (justify right bottom))
   )
@@
     (effects (font (size 1.27 1.27)) (justify right bottom))
   )
-  (label "B_IN" (at 60.96 111.76 0) (fields_autoplaced)
+  (label "B" (at 60.96 111.76 0) (fields_autoplaced)
     (effects (font (size 1.27 1.27)) (justify left bottom))
   )
@@
     (effects (font (size 1.27 1.27)) (justify right bottom))
   )
-  (label "R_IN" (at 60.96 91.44 0) (fields_autoplaced)
+  (label "R" (at 60.96 91.44 0) (fields_autoplaced)
     (effects (font (size 1.27 1.27)) (justify left bottom))
   )
@@
     )
   )
-  (symbol (lib_id "Device:C_Small") (at 132.08 44.45 0) (unit 1)
-    (in_bom yes) (on_board yes) (dnp no) (fields_autoplaced)
-    (property "Reference" "C10" (at 134.62 43.8213 0)
+  (symbol (lib_id "Device:C_Small") (at 132.08 44.45 0) (mirror y) (unit 1)
+    (in_bom yes) (on_board yes) (dnp no)
+    (property "Reference" "C10" (at 129.54 43.8213 0)
       (effects (font (size 1.27 1.27)) (justify left))
     )
-    (property "Value" "0.1u" (at 134.62 46.3613 0)
+    (property "Value" "0.1u" (at 129.54 46.3613 0)
       (effects (font (size 1.27 1.27)) (justify left))
     )
@@
   )
   (symbol (lib_id "REB_Transcoder:Connector_RCA_2x3_REB") (at 193.04 33.02 0) (unit 1)
-    (in_bom yes) (on_board yes) (dnp no)
-    (property "Reference" "J2" (at 212.09 44.45 0)
+    (in_bom yes) (on_board yes) (dnp no) (fields_autoplaced)
+    (property "Reference" "J2" (at 214.63 48.26 0)
       (effects (font (size 1.27 1.27)) (justify left))
     )
-    (property "Value" "Connector_RCA_2x3_REB" (at 212.09 46.99 0)
+    (property "Value" "Connector_RCA_2x3_REB" (at 214.63 50.8 0)
       (effects (font (size 1.27 1.27)) (justify left))
     )

Commit message: Minor tweaks
Parts:
- R5: value 680k -> 680K
- R6, R7: value 1k -> 1K
- R8, R9: value 2M2 -> 2.2M
Changed lines of the file:
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@@
       (effects (font (size 1.27 1.27)))
     )
-    (property "Value" "1k" (at 170.18 99.06 90)
+    (property "Value" "1K" (at 170.18 99.06 90)
       (effects (font (size 1.27 1.27)))
     )
@@
       (effects (font (size 1.27 1.27)) (justify right))
     )
-    (property "Value" "1k" (at 181.61 95.885 0)
+    (property "Value" "1K" (at 181.61 95.885 0)
       (effects (font (size 1.27 1.27)) (justify right))
     )
@@
       (effects (font (size 1.27 1.27)))
     )
-    (property "Value" "2M2" (at 179.07 144.78 90)
+    (property "Value" "2.2M" (at 179.07 144.78 90)
       (effects (font (size 1.27 1.27)))
     )
@@
       (effects (font (size 1.27 1.27)))
     )
-    (property "Value" "2M2" (at 179.07 124.46 90)
+    (property "Value" "2.2M" (at 179.07 124.46 90)
       (effects (font (size 1.27 1.27)))
     )
@@
       (effects (font (size 1.27 1.27)))
     )
-    (property "Value" "680k" (at 124.46 57.15 90)
-      (effects (font (size 1.27 1.27)))
-    )
+    (property "Value" "680K" (at 124.46 57.15 90)
+      (effects (font (size 1.27 1.27)))
+    )
